File: circuitos/led_potencia/led_potencia.kicad_pcb (KiCad board)
At the start: 2 copper layers, 12 parts, among them Q1 IRLZ44N, Q16 IRF4905, Q17 IRF4905, Q18 IRF4905, Q19 PN2222A, Q2 IRLZ44N, Q20 PN2222A, Q21 PN2222A, Q22 PN2222A, Q23 IRF4905, Q3 IRLZ44N, Q4 IRLZ44N

Commit message: mejorando array
Parts:
- added Q24: IRF4905, Package_TO_SOT_THT:TO-220-3_Vertical, F.Cu at (133.7, 108.4)
- added Q25: PN2222A, Package_TO_SOT_THT:TO-92_Inline, F.Cu at (107.5, 114.0)
- Q19, Q20: value PN2222A -> IRF4905; footprint Package_TO_SOT_THT:TO-92_Inline -> Package_TO_SOT_THT:TO-220-3_Vertical
- Q23: value IRF4905 -> PN2222A; footprint Package_TO_SOT_THT:TO-220-3_Vertical -> Package_TO_SOT_THT:TO-92_Inline
Connections:
- Q18 pad 3: unconnected-(Q18-S-Pad3) -> Net-(J1-Pin_2)
- Q19 pad 1: GND -> Net-(Q19-G)
- Q19 pad 2: Net-(Q19-B) -> +12V
- Q19 pad 3: Net-(Q16-G) -> Net-(J10-Pin_2)
- Q20 pad 1: GND -> Net-(Q20-G)
- Q20 pad 2: Net-(Q20-B) -> +12V
- Q20 pad 3: Net-(Q17-G) -> Net-(J11-Pin_2)
- Q22 pad 3: Net-(Q22-C) -> Net-(Q19-G)
- Q23 pad 1: Net-(Q22-C) -> GND
- Q23 pad 2: +12V -> Net-(Q23-B)
- Q23 pad 3: Net-(J1-Pin_2) -> Net-(Q20-G)
- Q4 pad 2: unconnected-(Q4-D-Pad2) -> Net-(J1-Pin_1)

Commit message: sumando cambios
Parts:
- removed Q16, Q17: IRF4905, Package_TO_SOT_THT:TO-220-3_Vertical
- added H1: MountingHole, MountingHole:MountingHole_2.2mm_M2_DIN965_Pad, F.Cu at (88.1, 57.6)
- added H2: MountingHole, MountingHole:MountingHole_2.2mm_M2_DIN965_Pad, F.Cu at (88.1, 62.9)
- added H3: MountingHole, MountingHole:MountingHole_2.2mm_M2_DIN965_Pad, F.Cu at (88.1, 68.3)
- added H4: MountingHole, MountingHole:MountingHole_2.2mm_M2_DIN965_Pad, F.Cu at (88.1, 73.6)
- added J1: Conn_01x02_Pin, Connector_Molex:Molex_KK-254_AE-6410-02A_1x02_P2.54mm_Vertical, F.Cu at (135.2, 19.6)
- added J10: Conn_01x02_Pin, Connector_Molex:Molex_KK-254_AE-6410-02A_1x02_P2.54mm_Vertical, F.Cu at (142.3, 35.3)
- added J11: Conn_01x02_Pin, Connector_Molex:Molex_KK-254_AE-6410-02A_1x02_P2.54mm_Vertical, F.Cu at (149.5, 35.3)
- added J12: Conn_01x02_Pin, Connector_Molex:Molex_KK-254_AE-6410-02A_1x02_P2.54mm_Vertical, F.Cu at (156.6, 35.3)
- added J13: Conn_01x02_Pin, Connector_Molex:Molex_KK-254_AE-6410-02A_1x02_P2.54mm_Vertical, F.Cu at (135.2, 43.2)
- added J14: Conn_01x02_Pin, Connector_Molex:Molex_KK-254_AE-6410-02A_1x02_P2.54mm_Vertical, F.Cu at (142.3, 43.2)
- added J15: Conn_01x02_Pin, Connector_Molex:Molex_KK-254_AE-6410-02A_1x02_P2.54mm_Vertical, F.Cu at (149.5, 43.2)
- added J16: Conn_01x02_Pin, Connector_Molex:Molex_KK-254_AE-6410-02A_1x02_P2.54mm_Vertical, F.Cu at (156.6, 43.2)
- added J17: Conn_01x02_Socket, Connector_Molex:Molex_KK-254_AE-6410-02A_1x02_P2.54mm_Vertical, F.Cu at (69.6, 155.9)
- added J18: Conn_01x02_Socket, Connector_Molex:Molex_KK-254_AE-6410-02A_1x02_P2.54mm_Vertical, F.Cu at (76.7, 155.9)
- added J2: Conn_01x02_Pin, Connector_Molex:Molex_KK-254_AE-6410-02A_1x02_P2.54mm_Vertical, F.Cu at (142.3, 19.6)
- added J3: Conn_01x02_Pin, Connector_Molex:Molex_KK-254_AE-6410-02A_1x02_P2.54mm_Vertical, F.Cu at (149.5, 19.6)
- added J4: Conn_01x02_Pin, Connector_Molex:Molex_KK-254_AE-6410-02A_1x02_P2.54mm_Vertical, F.Cu at (156.6, 19.6)
- added J5: Conn_01x02_Pin, Connector_Molex:Molex_KK-254_AE-6410-02A_1x02_P2.54mm_Vertical, F.Cu at (135.2, 27.5)
- added J6: Conn_01x02_Pin, Connector_Molex:Molex_KK-254_AE-6410-02A_1x02_P2.54mm_Vertical, F.Cu at (142.3, 27.5)
- added J7: Conn_01x02_Pin, Connector_Molex:Molex_KK-254_AE-6410-02A_1x02_P2.54mm_Vertical, F.Cu at (149.5, 27.5)
- added J8: Conn_01x02_Pin, Connector_Molex:Molex_KK-254_AE-6410-02A_1x02_P2.54mm_Vertical, F.Cu at (156.6, 27.5)
- added J9: Conn_01x02_Pin, Connector_Molex:Molex_KK-254_AE-6410-02A_1x02_P2.54mm_Vertical, F.Cu at (135.2, 35.3)
- added R1: 1k, Resistor_THT:R_Axial_DIN0309_L9.0mm_D3.2mm_P12.70mm_Horizontal, F.Cu at (178.2, 104.3)
- added R11: 10k, Resistor_THT:R_Axial_DIN0309_L9.0mm_D3.2mm_P12.70mm_Horizontal, F.Cu at (181.2, 35.8)
- added R12: 10k, Resistor_THT:R_Axial_DIN0309_L9.0mm_D3.2mm_P12.70mm_Horizontal, F.Cu at (186.0, 35.8)
- added R13: 10k, Resistor_THT:R_Axial_DIN0309_L9.0mm_D3.2mm_P12.70mm_Horizontal, F.Cu at (190.7, 35.8)
- added R14: 10k, Resistor_THT:R_Axial_DIN0309_L9.0mm_D3.2mm_P12.70mm_Horizontal, F.Cu at (195.5, 35.8)
- added R17: 10k, Resistor_THT:R_Axial_DIN0309_L9.0mm_D3.2mm_P12.70mm_Horizontal, F.Cu at (150.8, 73.0)
- added R18: 10k, Resistor_THT:R_Axial_DIN0309_L9.0mm_D3.2mm_P12.70mm_Horizontal, F.Cu at (167.2, 59.7)
- added R19: 10k, Resistor_THT:R_Axial_DIN0309_L9.0mm_D3.2mm_P12.70mm_Horizontal, F.Cu at (156.3, 59.6)
- added R2: 1k, Resistor_THT:R_Axial_DIN0309_L9.0mm_D3.2mm_P12.70mm_Horizontal, F.Cu at (172.4, 128.5)
- added R20: 10k, Resistor_THT:R_Axial_DIN0309_L9.0mm_D3.2mm_P12.70mm_Horizontal, F.Cu at (161.8, 72.2)
- added R3: 1k, Resistor_THT:R_Axial_DIN0309_L9.0mm_D3.2mm_P12.70mm_Horizontal, F.Cu at (164.8, 103.9)
- added R4: 1k, Resistor_THT:R_Axial_DIN0309_L9.0mm_D3.2mm_P12.70mm_Horizontal, F.Cu at (152.6, 103.7)
- added R5: 1k, Resistor_THT:R_Axial_DIN0309_L9.0mm_D3.2mm_P12.70mm_Horizontal, F.Cu at (173.7, 104.1)
- added R6: 1k, Resistor_THT:R_Axial_DIN0309_L9.0mm_D3.2mm_P12.70mm_Horizontal, F.Cu at (169.7, 104.0)
- added R7: 1k, Resistor_THT:R_Axial_DIN0309_L9.0mm_D3.2mm_P12.70mm_Horizontal, F.Cu at (160.8, 103.6)
- added R8: 1k, Resistor_THT:R_Axial_DIN0309_L9.0mm_D3.2mm_P12.70mm_Horizontal, F.Cu at (156.8, 103.6)
- added U1: 74HC595, Package_DIP:DIP-16_W7.62mm_Socket_LongPads, F.Cu at (174.9, 116.6)
- added puente1: 0, Resistor_THT:R_Axial_DIN0309_L9.0mm_D3.2mm_P15.24mm_Horizontal, F.Cu at (56.9, 25.9)
- added puente10: 0, Resistor_THT:R_Axial_DIN0309_L9.0mm_D3.2mm_P15.24mm_Horizontal, F.Cu at (56.9, 68.6)
- added puente11: 0, Resistor_THT:R_Axial_DIN0309_L9.0mm_D3.2mm_P15.24mm_Horizontal, F.Cu at (56.9, 73.4)
- added puente12: 0, Resistor_THT:R_Axial_DIN0309_L9.0mm_D3.2mm_P15.24mm_Horizontal, F.Cu at (56.9, 78.1)
- added puente2: 0, Resistor_THT:R_Axial_DIN0309_L9.0mm_D3.2mm_P15.24mm_Horizontal, F.Cu at (56.9, 30.6)
- added puente3: 0, Resistor_THT:R_Axial_DIN0309_L9.0mm_D3.2mm_P15.24mm_Horizontal, F.Cu at (56.9, 35.4)
- added puente4: 0, Resistor_THT:R_Axial_DIN0309_L9.0mm_D3.2mm_P15.24mm_Horizontal, F.Cu at (56.9, 40.1)
- added puente5: 0, Resistor_THT:R_Axial_DIN0309_L9.0mm_D3.2mm_P15.24mm_Horizontal, F.Cu at (56.9, 44.9)
- added puente6: 0, Resistor_THT:R_Axial_DIN0309_L9.0mm_D3.2mm_P15.24mm_Horizontal, F.Cu at (56.9, 49.6)
- added puente7: 0, Resistor_THT:R_Axial_DIN0309_L9.0mm_D3.2mm_P15.24mm_Horizontal, F.Cu at (56.9, 54.4)
- added puente8: 0, Resistor_THT:R_Axial_DIN0309_L9.0mm_D3.2mm_P15.24mm_Horizontal, F.Cu at (56.9, 59.1)
- added puente9: 0, Resistor_THT:R_Axial_DIN0309_L9.0mm_D3.2mm_P15.24mm_Horizontal, F.Cu at (56.9, 63.9)
- moved Q18 133.2 mm to (199.3, 64.0)
- moved Q22 119.4 mm to (208.1, 75.8), turned to 180 degrees
- moved Q25 116.2 mm to (217.4, 76.2), turned to 180 degrees
- moved Q23 116.0 mm to (185.0, 79.5)
- moved Q19 113.7 mm to (199.4, 51.0), turned to 180 degrees
- moved Q21 106.6 mm to (198.2, 82.7), turned to 180 degrees
- moved Q24 103.1 mm to (221.4, 54.2), turned to 180 degrees
- moved Q20 96.0 mm to (183.3, 64.1)
- moved Q1 93.5 mm to (173.7, 69.2), turned to 90 degrees
- moved Q2 33.6 mm to (108.7, 77.9)

Commit message: armando grilla PCB
Parts:
- puente1, puente10, puente11, puente12, puente2, puente3, puente4, puente5, puente6, puente7, puente8, puente9: footprint Resistor_THT:R_Axial_DIN0309_L9.0mm_D3.2mm_P15.24mm_Horizontal -> Resistor_THT:R_Axial_DIN0204_L3.6mm_D1.6mm_P5.08mm_Horizontal
- moved J17 149.7 mm to (216.5, 127.1), turned to -90 degrees
- moved puente12 145.9 mm to (200.1, 50.0), turned to 180 degrees
- moved Q24 94.0 mm to (153.3, 118.8), turned to 90 degrees
- moved R14 89.8 mm to (159.8, 118.3), turned to -90 degrees
- moved J18 89.7 mm to (163.5, 178.4), turned to 90 degrees
- moved Q25 88.2 mm to (154.0, 137.6), turned to 90 degrees
- moved Q1 86.8 mm to (109.5, 127.6), turned to 0 degrees
- moved R11 84.8 mm to (204.3, 117.5), turned to -90 degrees
- moved J1 83.3 mm to (199.5, 72.6), turned to 180 degrees
- moved R13 83.1 mm to (174.3, 117.3), turned to -90 degrees
- moved R12 81.0 mm to (188.3, 116.8), turned to -90 degrees
- moved J5 71.5 mm to (199.7, 58.3), turned to 180 degrees
- moved Q19 69.7 mm to (181.8, 118.4), turned to 90 degrees
- moved J2 67.1 mm to (183.5, 72.6), turned to 180 degrees
- moved Q22 66.8 mm to (183.9, 138.1), turned to 90 degrees
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
Commit message: circuito pre finalizado, retestear en proto e imprimir
Parts:
- removed J18: Conn_01x02_Socket, Connector_Molex:Molex_KK-254_AE-6410-02A_1x02_P2.54mm_Vertical
- added J19: Conn_01x02_OE_GND, Connector_Molex:Molex_KK-254_AE-6410-02A_1x02_P2.54mm_Vertical, F.Cu at (61.0, 122.5)
- added J20: Conn_01x05_Pin, Connector_Molex:Molex_KK-254_AE-6410-05A_1x05_P2.54mm_Vertical, F.Cu at (73.5, 141.0)
- added Puente_GND1: 0, Resistor_THT:R_Axial_DIN0204_L3.6mm_D1.6mm_P7.62mm_Horizontal, F.Cu at (62.4, 140.0)
- R1, R11, R12, R13, R14, R17, R18, R19, R2, R20, R3, R4, R5, R6, R7, R8: footprint Resistor_THT:R_Axial_DIN0309_L9.0mm_D3.2mm_P12.70mm_Horizontal -> Resistor_THT:R_Axial_DIN0204_L3.6mm_D1.6mm_P7.62mm_Horizontal
- moved R3 142.7 mm to (60.7, 37.0), turned to 0 degrees
- moved R7 125.9 mm to (60.7, 54.0), turned to 0 degrees
- moved H3 122.7 mm to (123.5, 142.5)
- moved R8 110.9 mm to (60.7, 69.5), turned to 0 degrees
- moved J17 108.8 mm to (107.8, 131.5), turned to 180 degrees
- moved R18 105.5 mm to (63.5, 41.5), turned to 0 degrees
- moved Q1 104.7 mm to (70.3, 30.5), turned to 180 degrees
- moved Q2 100.2 mm to (70.8, 47.5), turned to 180 degrees
- moved Q21 94.5 mm to (113.6, 103.3)
- moved R4 94.4 mm to (61.0, 87.0), turned to 0 degrees
- moved H2 94.0 mm to (123.5, 26.5)
- moved R20 93.4 mm to (71.3, 58.0), turned to 180 degrees
- moved R11 89.6 mm to (119.4, 88.7)
- moved Q22 88.2 mm to (102.9, 103.3)
- moved Q18 85.6 mm to (114.8, 93.0)
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Connections:
- R3 pad 1: Net-(U1-QE) -> Net-(U1-QH)
- R4 pad 1: Net-(U1-QH) -> Net-(U1-QE)
- R7 pad 1: Net-(U1-QF) -> Net-(U1-QG)
- R8 pad 1: Net-(U1-QG) -> Net-(U1-QF)
- U1 pad 10: unconnected-(U1-~{SRCLR}-Pad10) -> VCC
- U1 pad 11: unconnected-(U1-SRCLK-Pad11) -> Net-(J20-Pin_2)
- U1 pad 12: unconnected-(U1-RCLK-Pad12) -> Net-(J20-Pin_3)
- U1 pad 13: unconnected-(U1-~{OE}-Pad13) -> Net-(J19-Pin_2)
- U1 pad 14: unconnected-(U1-SER-Pad14) -> Net-(J20-Pin_4)
Routing:
- net GND: track 0.00 -> 366.8 mm
- net Net-(U1-QH): track 0.00 -> 96.2 mm
- net +12V: track 0.00 -> 95.7 mm
- net Net-(U1-QG): track 0.00 -> 77.8 mm
- net Net-(J13-Pin_1): track 0.00 -> 67.3 mm
- net Net-(U1-QF): track 0.00 -> 60.8 mm
- net Net-(J11-Pin_2): track 0.00 -> 58.9 mm
- net Net-(J1-Pin_2): track 0.00 -> 58.7 mm
- net Net-(J12-Pin_2): track 0.00 -> 58.6 mm
- net Net-(J10-Pin_2): track 0.00 -> 57.8 mm
- net VCC: track 0.00 -> 50.3 mm
- net Net-(U1-QA): track 0.00 -> 44.7 mm
- net Net-(U1-QE): track 0.00 -> 42.0 mm
- net Net-(U1-QB): track 0.00 -> 27.5 mm
- net Net-(J19-Pin_2): track 0.00 -> 21.0 mm
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- added copper zone on B.Cu, net GND
Other:
- board outline added: 84.5 x 128.5 mm

Commit message: in out añadidos
Parts:
- added J21: Conn_01x05_OUT, Connector_Molex:Molex_KK-254_AE-6410-05A_1x05_P2.54mm_Vertical, F.Cu at (79.5, 141.0)
- added Puente_OE1: 0, Resistor_THT:R_Axial_DIN0204_L3.6mm_D1.6mm_P5.08mm_Horizontal, F.Cu at (88.1, 137.0)
- J20: value Conn_01x05_Pin -> Conn_01x05_IN
- Puente_GND1: footprint Resistor_THT:R_Axial_DIN0204_L3.6mm_D1.6mm_P7.62mm_Horizontal -> Resistor_THT:R_Axial_DIN0207_L6.3mm_D2.5mm_P10.16mm_Horizontal
- moved Puente_GND1 32.0 mm to (93.1, 149.0), turned to 180 degrees
- moved H3 17.5 mm to (123.5, 160.0)
- moved H4 17.5 mm to (48.0, 160.5)
- moved J20 10.8 mm to (79.5, 150.0), turned to 180 degrees
- moved J17 9.12 mm to (99.0, 129.0)
Connections:
- U1 pad 11: Net-(J20-Pin_2) -> Net-(J20-Pin_3)
- U1 pad 12: Net-(J20-Pin_3) -> Net-(J20-Pin_2)
- U1 pad 13: Net-(J19-Pin_2) -> Net-(U1-~{OE})
- U1 pad 9: unconnected-(U1-QH'-Pad9) -> Net-(J21-Pin_4)
Routing:
- net Net-(J19-Pin_2): track 21.0 -> 73.0 mm
- net Net-(J20-Pin_4): track 12.4 -> 43.0 mm
- net Net-(J20-Pin_1): track 3.91 -> 22.2 mm
- net Net-(J21-Pin_4): track 0.00 -> 13.1 mm
- net Net-(U1-~{OE}): track 0.00 -> 9.47 mm
- net Net-(J20-Pin_3): track 12.7 -> 21.0 mm
- net Net-(J20-Pin_2): track 12.7 -> 21.0 mm
- net GND: track 366.8 -> 359.4 mm
- net Net-(U1-QA): track 44.7 -> 51.4 mm
- net +12V: track 95.7 -> 101.0 mm
- net VCC: track 50.3 -> 54.0 mm
- net Net-(Q20-G): track 13.3 -> 14.3 mm
- net Net-(J7-Pin_1): track 14.6 -> 15.3 mm
- net Net-(J6-Pin_1): track 14.7 -> 15.4 mm
- net Net-(Q24-G): track 13.1 -> 13.8 mm
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- removed copper zone on B.Cu, net GND
Other:
- board size 84.5 x 128.5 mm -> 84.5 x 145.5 mm

Commit message: variante de ruteo v2 contrastar?
Parts:
- moved J21 81.3 mm to (62.6, 61.5)
- moved J20 79.3 mm to (62.8, 72.5)
- moved J19 74.9 mm to (85.7, 51.8), turned to 180 degrees
- moved Puente_GND1 73.5 mm to (69.0, 79.6), turned to 90 degrees
- moved H4 66.5 mm to (58.0, 94.8)
- moved Puente_OE1 64.0 mm to (72.0, 75.0), turned to 90 degrees
- moved H3 62.6 mm to (159.5, 108.8)
- moved J17 60.3 mm to (150.4, 97.5), turned to -90 degrees
- moved U1 43.5 mm to (86.8, 77.9), turned to 180 degrees
- moved Q18 42.2 mm to (157.0, 92.0)
- moved R11 42.2 mm to (161.7, 87.7)
- moved R13 35.5 mm to (132.6, 88.5)
- moved R4 35.5 mm to (96.5, 86.8)
- moved H2 35.5 mm to (159.0, 26.3)
- moved J10 35.5 mm to (141.3, 43.2)
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Routing:
- net GND: track 359.4 -> 270.2 mm
- net Net-(U1-QH): track 96.2 -> 30.2 mm
- net Net-(U1-QG): track 77.8 -> 17.1 mm
- net Net-(U1-QF): track 60.8 -> 10.0 mm
- net +12V: track 101.0 -> 62.9 mm
- net Net-(U1-QB): track 27.5 -> 63.6 mm
- net Net-(U1-QA): track 51.4 -> 84.5 mm
- net VCC: track 54.0 -> 80.4 mm
- net Net-(U1-QC): track 19.1 -> 43.3 mm
- net Net-(J20-Pin_3): track 21.0 -> 43.8 mm
- net Net-(J21-Pin_4): track 13.1 -> 34.8 mm
- net Net-(U1-QE): track 42.0 -> 23.8 mm
- net Net-(J20-Pin_2): track 21.0 -> 39.0 mm
- net Net-(J20-Pin_4): track 43.0 -> 27.7 mm
- net Net-(U1-QD): track 14.6 -> 27.4 mm
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Other:
- board size 84.5 x 145.5 mm -> 131.2 x 95.8 mm

Commit message: obse nomai v3 de ruteo (podria achicarse mucho mas pero no es sano
Parts:
- moved Puente_GND1 31.5 mm to (62.0, 48.8), turned to -90 degrees
- moved H1 9.30 mm to (62.2, 33.5)
- moved J20 8.53 mm to (67.0, 65.1), turned to -90 degrees
- moved J21 4.98 mm to (67.0, 59.1), turned to 90 degrees
- moved H3 3.78 mm to (160.0, 105.0)
- moved R1 1.46 mm to (128.2, 107.3)
Routing:
- net GND: track 270.2 -> 206.0 mm
- net Net-(J21-Pin_4): track 34.8 -> 15.9 mm
- net Net-(J20-Pin_4): track 27.7 -> 12.3 mm
- net Net-(J20-Pin_2): track 39.0 -> 25.4 mm
- net VCC: track 80.4 -> 84.8 mm
- net Net-(J20-Pin_1): track 21.6 -> 17.4 mm
- net Net-(Q22-B): track 4.13 -> 7.26 mm
- net Net-(U1-QH): track 30.2 -> 31.5 mm
- net Net-(J19-Pin_2): track 85.4 -> 86.7 mm
- net Net-(U1-QB): track 63.6 -> 62.5 mm
- net Net-(U1-QA): track 84.5 -> 83.5 mm
- net Net-(U1-QG): track 17.1 -> 17.9 mm
Other:
- board size 131.2 x 95.8 mm -> 115.2 x 91.5 mm
