File: circuitos/led_potencia/led_potencia.kicad_pcb (KiCad board)
At the start: 2 copper layers, 115.2 x 91.5 mm, 67 parts, among them J1 Conn_01x02_Pin, J10 Conn_01x02_Pin, J11 Conn_01x02_Pin, J12 Conn_01x02_Pin, J13 Conn_01x02_Pin, J14 Conn_01x02_Pin, J15 Conn_01x02_Pin, J16 Conn_01x02_Pin, J17 Conn_01x02_Socket, J19 Conn_01x02_OE_GND, J2 Conn_01x02_Pin, J20 Conn_01x05_IN, J21 Conn_01x05_OUT, J3 Conn_01x02_Pin, J4 Conn_01x02_Pin, J5 Conn_01x02_Pin, J6 Conn_01x02_Pin, J7 Conn_01x02_Pin, J8 Conn_01x02_Pin, J9 Conn_01x02_Pin, Q1 IRLZ44N, Q18 IRF4905, Q19 IRF4905, Q2 IRLZ44N, Q20 IRF4905, Q21 PN2222A, Q22 PN2222A, Q23 PN2222A, Q24 IRF4905, Q25 PN2222A, Q3 IRLZ44N, Q4 IRLZ44N, U1 74HC595

Commit message: holes
Parts:
- moved H4 12.5 mm to (56.7, 107.2)
- moved H1 8.23 mm to (56.7, 27.4)
- moved H3 2.19 mm to (160.0, 107.2)
- moved H2 1.45 mm to (160.0, 27.4)
Changed lines of the file:
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@@
 	(footprint "MountingHole:MountingHole_2.2mm_M2_DIN965_Pad"
 		(layer "F.Cu")
-		(at 58 94.75)
+		(at 56.7436 107.188)
 		(descr "Mounting Hole 2.2mm, M2, generated by kicad-footprint-generator mountinghole.py")
 		(tags "mountinghole M2 DIN965")
@@
 	(footprint "MountingHole:MountingHole_2.2mm_M2_DIN965_Pad"
 		(layer "F.Cu")
-		(at 159.03 26.27)
+		(at 159.9692 27.3812)
 		(descr "Mounting Hole 2.2mm, M2, generated by kicad-footprint-generator mountinghole.py")
 		(tags "mountinghole M2 DIN965")
@@
 	(footprint "MountingHole:MountingHole_2.2mm_M2_DIN965_Pad"
 		(layer "F.Cu")
-		(at 62.25 33.5)
+		(at 56.7436 27.3812)
 		(descr "Mounting Hole 2.2mm, M2, generated by kicad-footprint-generator mountinghole.py")
 		(tags "mountinghole M2 DIN965")
@@
 	(footprint "MountingHole:MountingHole_2.2mm_M2_DIN965_Pad"
 		(layer "F.Cu")
-		(at 160 105)
+		(at 159.9692 107.188)
 		(descr "Mounting Hole 2.2mm, M2, generated by kicad-footprint-generator mountinghole.py")
 		(tags "mountinghole M2 DIN965")
