File: circuitos/led_potencia/led_potencia.kicad_pcb (KiCad board)
At the start: 2 copper layers, 44 parts, among them J1 Conn_01x03_Pin, J10 Conn_01x02_Pin, J11 Conn_01x02_Pin, J12 Conn_01x02_Pin, J13 Conn_01x02_Pin, J14 Conn_01x02_Pin, J15 Conn_01x02_Pin, J16 Conn_01x02_Pin, J17 Conn_01x02_Socket, J18 Conn_01x02_Socket, J19 Conn_01x02_Socket, J2 Conn_01x03_Pin, J20 Conn_01x05_IN, J21 Conn_01x05_OUT, J9 Conn_01x02_Pin, Q17 IRLZ44N, Q18 IRLZ44N, Q19 IRLZ44N, Q20 IRLZ44N, Q21 IRLZ44N, Q22 IRLZ44N, Q23 IRLZ44N, Q24 IRLZ44N, U1 74HC595

Commit message: ruteo : pre inversion
Parts:
- removed J20: Conn_01x05_IN, Connector_Molex:Molex_KK-254_AE-6410-05A_1x05_P2.54mm_Vertical
- removed J21: Conn_01x05_OUT, Connector_Molex:Molex_KK-254_AE-6410-05A_1x05_P2.54mm_Vertical
- added J3: Conn_01x02_Socket, Connector_Molex:Molex_KK-254_AE-6410-02A_1x02_P2.54mm_Vertical, F.Cu at (171.5, 23.0)
- added puente1: 0, Resistor_THT:R_Axial_DIN0204_L3.6mm_D1.6mm_P7.62mm_Horizontal, F.Cu at (159.0, 56.8)
- moved H3 151.5 mm to (141.5, 21.5)
- moved H1 124.1 mm to (136.0, 84.0)
- moved J19 123.0 mm to (171.5, 31.0), turned to 180 degrees
- moved H2 108.0 mm to (201.5, 21.5)
- moved Q24 59.3 mm to (153.9, 67.9), turned to 0 degrees
- moved J17 57.5 mm to (145.0, 56.0), turned to 180 degrees
- moved J16 56.0 mm to (156.5, 75.3), turned to 90 degrees
- moved R9 53.2 mm to (159.2, 59.6), turned to 180 degrees
- moved H4 52.5 mm to (224.0, 84.0)
- moved J9 50.9 mm to (179.5, 22.8), turned to -90 degrees
- moved R40 50.8 mm to (160.4, 62.6), turned to 180 degrees
- moved J18 46.2 mm to (146.5, 63.0), turned to -90 degrees
- moved Q17 45.4 mm to (182.3, 29.5), turned to 180 degrees
- moved R33 41.1 mm to (183.3, 34.8), turned to 180 degrees
- moved R39 40.0 mm to (164.7, 69.0), turned to 0 degrees
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Connections:
- J17 pad 1: +12V -> GND
- J17 pad 2: GND -> +12V
- J18 pad 1: +12V -> GND
- J18 pad 2: GND -> +12V
- J19 pad 1: VCC -> GND
- J19 pad 2: Net-(J19-Pin_2) -> VCC
Routing:
- net GND: track 12.2 -> 217.4 mm
- net +12V: track 0.00 -> 147.0 mm
- net VCC: track 0.00 -> 41.7 mm
- net Net-(J1-Pin_3): track 0.00 -> 33.4 mm
- net Net-(J1-Pin_2): track 0.00 -> 18.6 mm
- net Net-(J1-Pin_1): track 0.00 -> 18.6 mm
- net Net-(U1-QD): track 0.00 -> 16.8 mm
- net Net-(J2-Pin_3): track 0.00 -> 11.5 mm
- net Net-(U1-QC): track 0.00 -> 11.4 mm
- net Net-(Q21-G): track 0.00 -> 10.5 mm
- net Net-(Q22-G): track 0.00 -> 9.66 mm
- net Net-(Q20-G): track 0.00 -> 9.61 mm
- net Net-(U1-QB): track 0.00 -> 9.30 mm
- net Net-(Q24-G): track 0.00 -> 9.26 mm
- net Net-(U1-QE): track 0.00 -> 9.14 mm
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
Commit message: ruteo : pre inversion
Parts:
- J1, J10, J11, J12, J13, J14, J15, J16, J17, J18, J19, J2, J3, J9, Q17, Q18, Q19, Q20, Q21, Q22, Q23, Q24, R10, R11, R12, R13, R14, R15, R16, R33, R34, R35, R36, R37, R38, R39, R40, R9, U1, puente1: moved to B.Cu
- moved J11 61.8 mm to (141.2, 44.0), turned to 0 degrees
- moved J10 57.4 mm to (143.4, 32.3), turned to 0 degrees
- moved J12 57.3 mm to (143.4, 54.9), turned to 0 degrees
- moved J17 54.2 mm to (199.2, 56.0), turned to 0 degrees
- moved J13 52.4 mm to (145.9, 67.5), turned to 0 degrees
- moved J1 52.2 mm to (198.2, 44.5)
- moved J18 51.2 mm to (197.7, 63.0)
- moved Q19 48.0 mm to (148.1, 46.2)
- moved Q20 43.7 mm to (150.2, 57.5)
- moved Q18 43.3 mm to (150.4, 34.9)
- moved Q21 38.8 mm to (152.7, 70.0)
- moved R35 36.8 mm to (153.7, 47.8)
- moved Q24 36.3 mm to (190.3, 67.9), turned to 180 degrees
- moved J2 36.2 mm to (190.2, 44.4)
- moved R34 31.8 mm to (156.2, 28.7)
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Routing:
- added copper zone on B.Cu, net GND
Other:
- board outline added: 69 x 73 mm
