File: circuitos/led_potencia/led_potencia.kicad_sch (KiCad schematic)
At the start: 67 parts, among them J1 Conn_01x02_Pin, J10 Conn_01x02_Pin, J11 Conn_01x02_Pin, J12 Conn_01x02_Pin, J13 Conn_01x02_Pin, J14 Conn_01x02_Pin, J15 Conn_01x02_Pin, J16 Conn_01x02_Pin, J17 Conn_01x02_Socket, J19 Conn_01x02_OE_GND, J2 Conn_01x02_Pin, J20 Conn_01x05_IN, J21 Conn_01x05_OUT, J3 Conn_01x02_Pin, J4 Conn_01x02_Pin, J5 Conn_01x02_Pin, J6 Conn_01x02_Pin, J7 Conn_01x02_Pin, J8 Conn_01x02_Pin, J9 Conn_01x02_Pin, Q1 IRLZ44N, Q18 IRF4905, Q19 IRF4905, Q2 IRLZ44N, Q20 IRF4905, Q21 PN2222A, Q22 PN2222A, Q23 PN2222A, Q24 IRF4905, Q25 PN2222A, Q3 IRLZ44N, Q4 IRLZ44N, U1 74HC595

Commit message: problemas tecnicos prueba y notas sobre circuito correcto sobre proto
Other:
- note added: "INVERTIR EN LA PCB LOS IRF Y LOS 2n2222"
- note added: "PARECEN ESTAR BIEN"
- note added: "agregar 1k Resis"
- note added: "revision en protoboard 5v y señales activas de irlz44n y 2n2222 a 3.3: IRLZ44N gate ( pin 1) 10k a pull Down 1k a señal (vcc activa el paso de corriente) drain ( pin 2) a gnd-terminal source (pin 3) a GND IRF9630 gate ( pin 1) 10k a pull up 1k a señal (gnd activa el paso de corriente)(2n2222) drain ( pin 2) a Vout-terminal source (pin 3) a VIN 2n2222 emisor (pin 1)( señal hacia irf9630 via 1k res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"
- moved on the sheet: Q19, Q20, Q21, Q22, Q23, Q25

Commit message: todo: ruteo y revision de pcb ya impreso en funcion de porque no prende y apaga
Connections:
- net +12V: now also Q18.3 (S), Q19.3 (S), Q20.3 (S), Q24.3 (S); no longer Q18.2 (D), Q19.2 (D), Q20.2 (D), Q24.2 (D)
- net at J10.2 (Pin_2), J14.2 (Pin_2), J2.2 (Pin_2)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: now also Q19.2 (D); no longer Q19.3 (S)
- net at J11.2 (Pin_2), J15.2 (Pin_2), J3.2 (Pin_2)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: now also Q20.2 (D); no longer Q20.3 (S)
- net at J12.2 (Pin_2), J16.2 (Pin_2), J4.2 (Pin_2)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: now also Q24.2 (D); no longer Q24.3 (S)
- net at J1.2 (Pin_2), J13.2 (Pin_2), J5.2 (Pin_2)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: now also Q18.2 (D); no longer Q18.3 (S)
Other:
- note added: "revision en protoboard 5v y señales activas de irlz44n y 2n2222 a 3.3: IRLZ44N gate ( pin 1) 10k a pull Down 1k a señal (vcc activa el paso de corriente) drain ( pin 2) a gnd-terminal source (pin 3) a GND IRF9630 gate ( pin 1) 10k a pull up 1k a señal (gnd activa el paso de corriente)(2n2222) drain ( pin 2) a Vout-terminal source (pin 3) a VIN 2n2222 emisor (pin 1)a GND base (pin 2) señal ic ( vi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"
- note removed: "INVERTIR EN LA PCB LOS IRF Y LOS 2n2222"
- note removed: "revision en protoboard 5v y señales activas de irlz44n y 2n2222 a 3.3: IRLZ44N gate ( pin 1) 10k a pull Down 1k a señal (vcc activa el paso de corriente) drain ( pin 2) a gnd-terminal source (pin 3) a GND IRF9630 gate ( pin 1) 10k a pull up 1k a señal (gnd activa el paso de corriente)(2n2222) drain ( pin 2) a Vout-terminal source (pin 3) a VIN 2n2222 emisor (pin 1)( señal hacia irf9630 via 1k res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"
- moved on the sheet: Q18, Q19, Q20, Q24
Changed lines of the file:
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@@
 	(generator_version "10.0")
 	(paper "A4")
-	(text "\nrevision en protoboard 5v y señales activas de irlz44n y 2n2222 a 3.3:\nIRLZ44N\ngate ( pin 1) 10k a pull Down 1k a señal (vcc activa el paso de corriente)\ndrain ( pin 2) a gnd-terminal\nsource (pin 3) a GND\n\nIRF9630\ngate ( pin 1) 10k a pull up 1k a señal (gnd activa el paso de corriente)(2n2222)\ndrain ( pin 2) a Vout-terminal\nsource (pin 3) a VIN\n\n2n2222\nemisor (pin 1)( señal hacia irf9630 via 1k resi) vcc activa el paso de corriente)\nbase (pin 2) señal ic ( via 1k Resi)\ncolector (pin 3) a GND"
+	(text "\nrevision en protoboard 5v y señales activas de irlz44n y 2n2222 a 3.3:\nIRLZ44N\ngate ( pin 1) 10k a pull Down 1k a señal (vcc activa el paso de corriente)\ndrain ( pin 2) a gnd-terminal\nsource (pin 3) a GND\n\nIRF9630\ngate ( pin 1) 10k a pull up 1k a señal (gnd activa el paso de corriente)(2n2222)\ndrain ( pin 2) a Vout-terminal\nsource (pin 3) a VIN\n\n2n2222\nemisor (pin 1)a GND \nbase (pin 2) señal ic ( via 1k Resi)\ncolector (pin 3) a  señal hacia irf9630 (via 1k resi idealmente) vcc activa el paso de corriente)"
 		(exclude_from_sim no)
 		(at 20.574 17.272 0)
@@
 		(exclude_from_sim no)
 		(at 216.916 171.704 0)
-		(effects
-			(font
-				(size 1.27 1.27)
-			)
-		)
-	)
-	(text "INVERTIR EN LA PCB LOS IRF Y LOS 2n2222\n"
-		(exclude_from_sim no)
-		(at 147.32 22.606 0)
 		(effects
 			(font
@@
 	(symbol
 		(lib_id "Transistor_FET:IRF4905")
-		(at 132.08 57.15 90)
+		(at 132.08 57.15 270)
+		(mirror x)
 		(unit 1)
 		(body_style 1)
@@
 		(in_pos_files yes)
 		(dnp no)
-		(fields_autoplaced yes)
 		(property "Reference" "Q19"
-			(at 130.8099 50.8 0)
+			(at 133.3501 50.8 0)
 			(show_name no)
 			(do_not_autoplace no)
@@
 		)
 		(property "Value" "IRF4905"
-			(at 133.3499 50.8 0)
+			(at 130.8101 50.8 0)
 			(show_name no)
 			(do_not_autoplace no)
@@
 		)
 		(property "Footprint" "Package_TO_SOT_THT:TO-220-3_Vertical"
-			(at 133.985 52.07 0)
+			(at 130.175 52.07 0)
 			(hide yes)
 			(show_name no)
@@
 		)
 		(property "Datasheet" "http://www.infineon.com/dgdl/irf4905.pdf?fileId=5546d462533600a4015355e32165197c"
-			(at 135.89 52.07 0)
+			(at 128.27 52.07 0)
 			(hide yes)
 			(show_name no)
@@
 	(symbol
 		(lib_id "Transistor_FET:IRF4905")
-		(at 133.35 76.2 90)
+		(at 133.35 76.2 270)
+		(mirror x)
 		(unit 1)
 		(body_style 1)
@@
 		(dnp no)
 		(property "Reference" "Q20"
-			(at 140.9699 69.85 0)
+			(at 125.7301 69.85 0)
 			(show_name no)
 			(do_not_autoplace no)
@@
 		)
 		(property "Value" "IRF4905"
-			(at 143.5099 69.85 0)
+			(at 123.1901 69.85 0)
 			(show_name no)
 			(do_not_autoplace no)
@@
 		)
 		(property "Footprint" "Package_TO_SOT_THT:TO-220-3_Vertical"
-			(at 135.255 71.12 0)
+			(at 131.445 71.12 0)
 			(hide yes)
 			(show_name no)
@@
 		)
 		(property "Datasheet" "http://www.infineon.com/dgdl/irf4905.pdf?fileId=5546d462533600a4015355e32165197c"
-			(at 137.16 71.12 0)
+			(at 129.54 71.12 0)
 			(hide yes)
 			(show_name no)
@@
 	(symbol
 		(lib_id "Transistor_FET:IRF4905")
-		(at 128.27 93.98 90)
+		(at 128.27 93.98 270)
+		(mirror x)
 		(unit 1)
 		(body_style 1)
@@
 		(in_pos_files yes)
 		(dnp no)
-		(fields_autoplaced yes)
 		(property "Reference" "Q24"
-			(at 126.9999 87.63 0)
+			(at 129.5401 87.63 0)
 			(show_name no)
 			(do_not_autoplace no)
@@
 		)
 		(property "Value" "IRF4905"
-			(at 129.5399 87.63 0)
+			(at 127.0001 87.63 0)
 			(show_name no)
 			(do_not_autoplace no)
@@
 		)
 		(property "Footprint" "Package_TO_SOT_THT:TO-220-3_Vertical"
-			(at 130.175 88.9 0)
+			(at 126.365 88.9 0)
 			(hide yes)
 			(show_name no)
@@
 		)
 		(property "Datasheet" "http://www.infineon.com/dgdl/irf4905.pdf?fileId=5546d462533600a4015355e32165197c"
-			(at 132.08 88.9 0)
+			(at 124.46 88.9 0)
 			(hide yes)
 			(show_name no)
@@
 	(symbol
 		(lib_id "Transistor_FET:IRF4905")
-		(at 123.19 31.75 90)
+		(at 123.19 31.75 270)
+		(mirror x)
 		(unit 1)
 		(body_style 1)
@@
 		(in_pos_files yes)
 		(dnp no)
-		(fields_autoplaced yes)
 		(property "Reference" "Q18"
-			(at 121.9199 25.4 0)
+			(at 124.4601 25.4 0)
 			(show_name no)
 			(do_not_autoplace no)
@@
 		)
 		(property "Value" "IRF4905"
-			(at 124.4599 25.4 0)
+			(at 121.9201 25.4 0)
 			(show_name no)
 			(do_not_autoplace no)
@@
 		)
 		(property "Footprint" "Package_TO_SOT_THT:TO-220-3_Vertical"
-			(at 125.095 26.67 0)
+			(at 121.285 26.67 0)
 			(hide yes)
 			(show_name no)
@@
 		)
 		(property "Datasheet" "http://www.infineon.com/dgdl/irf4905.pdf?fileId=5546d462533600a4015355e32165197c"
-			(at 127 26.67 0)
-			(hide yes)
-			(show_name no)
+			(at 119.38 26.67 0)
+			(hide yes)
+			(show_name no)
